File: Sega Genesis Cartridge/Sega Genesis Cartridge.sch (KiCad schematic (older format))
At the start: 4 parts

Commit message: Circuit schematic rev A
Parts:
- removed J?: Side B, symbol Connector_Generic:Conn_01x32
- removed J?: Side A, symbol Connector_Generic:Conn_01x32
- removed U? (x2): SST39SF040, symbol Memory_Flash:SST39SF040
- added C1: CP, symbol Device:CP
- added C2, C3: C, symbol Device:C
- added J1: Side A, symbol Genesis_Cart:cart_edge_conn_side_A
- added J2: Side B, symbol Genesis_Cart:cart_edge_conn_side_B
- added SW1: my_SW_SP3T, symbol Genesis_Cart:my_SW_SP3T
- added U1, U2: my_SST39SF040, symbol Genesis_Cart:my_SST39SF040
Connections:
- net labels added: A10, A18, A19, A9, VCC, ~CART, ~CAS0, ~CE, ~CEO, ~OE, ~WE
- wire segments 48 -> 137
Other:
- note added: "* A1 is the first address bit. Bit 0 is hardwired low."
- note added: "* External programmer can use ~WE.\n Console pulls the pin high."
- note added: "2-1 4 Mbit Low\n2-3 8 Mbit\n2-4 4 Mbit High\n"
- note added: "Bypass capacitors"
- note added: "Edge Connector"

Commit message: Capacitor values
Parts:
- C1: value CP -> 47 uF
- C2, C3: value C -> 0.1 uF
Changed lines of the file:
@@
 P 1400 1125
 F 0 "C1" H 1518 1171 50  0000 L CNN
-F 1 "CP" H 1518 1080 50  0000 L CNN
+F 1 "47 uF" H 1518 1080 50  0000 L CNN
 F 2 "" H 1438 975 50  0001 C CNN
 F 3 "~" H 1400 1125 50  0001 C CNN
@@
 P 5500 6755
 F 0 "C3" H 5615 6801 50  0000 L CNN
-F 1 "C" H 5615 6710 50  0000 L CNN
+F 1 "0.1 uF" H 5615 6710 50  0000 L CNN
 F 2 "" H 5538 6605 50  0001 C CNN
 F 3 "~" H 5500 6755 50  0001 C CNN
@@
 P 5000 6750
 F 0 "C2" H 5115 6796 50  0000 L CNN
-F 1 "C" H 5115 6705 50  0000 L CNN
+F 1 "0.1 uF" H 5115 6705 50  0000 L CNN
 F 2 "" H 5038 6600 50  0001 C CNN
 F 3 "~" H 5000 6750 50  0001 C CNN

Commit message: Begin PCB layout
Revised schematic, added footprints and strated PCB layout.
Parts:
- removed J1: Side A, symbol Genesis_Cart:cart_edge_conn_side_A
- removed J2: Side B, symbol Genesis_Cart:cart_edge_conn_side_B
- added J1: edge_connector, Genesis_Cart:Genesis_cart_edge_connector, symbol Genesis_Cart:cart_edge_conn_double_sided
- C1, C2, C3: footprint (none) -> Capacitors_SMD:C_0805_HandSoldering
- SW1: footprint (none) -> Genesis_Cart:MHS_133_Series_Switch
- U1, U2: footprint (none) -> SMD_Packages:TSOP32SP
Connections:
- net labels removed: ~CAS0, ~CEO
- wire segments 137 -> 138
Other:
- moved on the sheet: C1
