File: Sega Genesis Flash Cart/Sega Genesis Flash Cart.sch (KiCad schematic (older format))
At the start: 7 parts, among them J1 edge_connector, SW1 my_SW_SP3T, U1 my_SST39SF040, U2 my_SST39SF040

Commit message: Revised PCB and schematic
Changed schematic symbol for Genesis edge connector.
 Changed footprint for Genesis edge connector.  Ripped all traces and re-routed the PCB.
Parts:
- removed J1: edge_connector, Genesis_Cart:Genesis_cart_edge_connector, symbol Sega-Genesis-Cartridge-rescue:cart_edge_conn_double_sided-Genesis_Cart
- removed SW1: my_SW_SP3T, Genesis_Cart:MHS_133_Series_Switch, symbol Sega-Genesis-Cartridge-rescue:my_SW_SP3T-Genesis_Cart
- removed U1, U2: my_SST39SF040, Package_DIP:DIP-32_W15.24mm, symbol Sega-Genesis-Cartridge-rescue:my_SST39SF040-Genesis_Cart
- added J1: Sega_Genesis_Cart_Edge_Connector, Sega_Genesis_Cart:GENESIS-EDGE, symbol Sega_Genesis_Flash_Cart:Sega_Genesis_Cart_Edge_Connector
- added SW1: SW_SP3T, Sega_Genesis_Cart:MHS_133_Series_Switch, symbol Sega_Genesis_Flash_Cart:SW_SP3T
- added U1, U2: SST39SF040, Package_DIP:DIP-32_W15.24mm, symbol Sega_Genesis_Flash_Cart:SST39SF040
Connections:
- net labels added: BANK
- wire segments 138 -> 133
- no-connect marks 0 -> 1
Other:
- note added: "Bank Selector\n2-1 4 Mbit Low\n2-3 8 Mbit\n2-4 4 Mbit High\n"
- note removed: "* External programmer can use ~WE.\n Console pulls the pin high."
- note removed: "2-1 4 Mbit Low\n2-3 8 Mbit\n2-4 4 Mbit High\n"
- moved on the sheet: C1
